File: schematics/src/mainboard/mainboard.brd (EAGLE design)
At the start: 48.3 x 99.7 mm, 58 parts, among them IC1 CEM3320, IC2 ADG412N, IC3 ADG412N, IC6 78L05Z, IC7 TL072P, Q1 BC559C

Commit message: Faceplates & Bugfixes
Parts:
- C1, C2, C3, C7: device resistor:C050-024X044 -> rcl:C050-050X075
- moved C2 8.64 mm to (3.17, 24.8), turned to 270 degrees
- moved C10 5.12 mm to (3.17, 33.7), turned to 90 degrees
- moved C9 2.01 mm to (4.45, 40.6)
- moved C7 2.01 mm to (36.8, 34.3)
- moved C3 1.42 mm to (36.8, 28.6)
- moved D2 1.27 mm to (12.7, 24.8)
- moved R10 1.27 mm to (12.7, 19.7)
- moved R6 1.27 mm to (12.7, 22.2)
- moved PWR 1.27 mm to (35.6, 5.08)
- moved R7 1.27 mm to (36.8, 38.7)
- moved R5 0.64 mm to (36.8, 24.1)
- moved C4 0.63 mm to (43.2, 14.6)
- moved C5 0.63 mm to (36.2, 14.6)
Routing:
- net N$26: track 6.35 -> 17.1 mm
- net P17: track 48.7 -> 40.9 mm, vias 0 -> 1
- net P2: track 78.9 -> 75.9 mm
- net N$6: track 41.4 -> 39.3 mm
- net P18: track 42.1 -> 40.3 mm
- net P7: track 29.6 -> 31.4 mm
- net N$9: track 40.7 -> 42.2 mm
- net P5: track 5.71 -> 6.98 mm
- net P10: track 84.3 -> 83.1 mm
- net INT_RES: track 65.8 -> 64.5 mm
- net P4: track 5.71 -> 6.88 mm
- net N$1: track 49.9 -> 48.8 mm
- net P1: track 33.0 -> 33.8 mm
- net +12V: track 197.0 -> 197.5 mm
- net P6: track 83.5 -> 84.0 mm
Other:
- board text added: "+12v"
- board text added: "-12v"
- board text added: "Elka Synthex VCF Clone 1.2 gerbster.nl 2022"
- board text removed: "Elka Synthex VCF Clone gerbster.nl 2020"
