File: schematics/src/mainboard/mainboard.sch (EAGLE design)
At the start: 58 parts, among them IC1 CEM3320, IC2 ADG412N, IC3 ADG412N, IC6 78L05Z, IC7 TL072P, Q1 BC559C

Commit message: Faceplates & Bugfixes
Parts:
- C1, C2, C3, C7: device resistor:C-EU050-024X044 -> rcl:C-EU050-050X075
Changed lines of the file:
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@@
 <part name="R1" library="resistor" deviceset="R-US_" device="0207/10" value="1.2k"/>
 <part name="GND2" library="supply1" deviceset="GND" device=""/>
-<part name="C1" library="resistor" deviceset="C-EU" device="050-024X044" value="330pf"/>
-<part name="C2" library="resistor" deviceset="C-EU" device="050-024X044" value="330pf"/>
+<part name="C1" library="rcl" library_urn="urn:adsk.eagle:library:334" deviceset="C-EU" device="050-050X075" package3d_urn="urn:adsk.eagle:package:23665/1" value="330pf"/>
+<part name="C2" library="rcl" library_urn="urn:adsk.eagle:library:334" deviceset="C-EU" device="050-050X075" package3d_urn="urn:adsk.eagle:package:23665/1" value="330pf"/>
 <part name="GND4" library="supply1" deviceset="GND" device=""/>
 <part name="R4" library="pot" deviceset="TRIM_1234-" device="S64YW" value="10k"/>
@@
 <part name="P+2" library="supply1" deviceset="+12V" device=""/>
 <part name="R17" library="resistor" deviceset="R-US_" device="0207/10" value="10k"/>
-<part name="C3" library="resistor" deviceset="C-EU" device="050-024X044" value="330pf"/>
+<part name="C3" library="rcl" library_urn="urn:adsk.eagle:library:334" deviceset="C-EU" device="050-050X075" package3d_urn="urn:adsk.eagle:package:23665/1" value="330pf"/>
 <part name="GND6" library="supply1" deviceset="GND" device=""/>
 <part name="C6" library="resistor" deviceset="CPOL-US" device="E2.5-5" value="4.7uf/50v"/>
 <part name="R18" library="resistor" deviceset="R-US_" device="0207/10" value="68k"/>
-<part name="C7" library="resistor" deviceset="C-EU" device="050-024X044" value="330pf"/>
+<part name="C7" library="rcl" library_urn="urn:adsk.eagle:library:334" deviceset="C-EU" device="050-050X075" package3d_urn="urn:adsk.eagle:package:23665/1" value="330pf"/>
 <part name="R19" library="resistor" deviceset="R-US_" device="0207/10" value="10k"/>
 <part name="GND7" library="supply1" deviceset="GND" device=""/>
@@
 </schematic>
 </drawing>
+<compatibility>
+<note version="8.2" severity="warning">
+Since Version 8.2, EAGLE supports online libraries. The ids
+of those online libraries will not be understood (or retained)
+with this version.
+</note>
+<note version="8.3" severity="warning">
+Since Version 8.3, EAGLE supports URNs for individual library
+assets (packages, symbols, and devices). The URNs of those assets
+will not be understood (or retained) with this version.
+</note>
+<note version="8.3" severity="warning">
+Since Version 8.3, EAGLE supports the association of 3D packages
+with devices in libraries, schematics, and board files. Those 3D
+packages will not be understood (or retained) with this version.
+</note>
+<note version="8.4" severity="warning">
+Since Version 8.4, EAGLE supports properties for SPICE simulation.
+Probes in schematics and SPICE mapping objects found in parts and library devices
+will not be understood with this version. Update EAGLE to the latest version
+for full support of SPICE simulation.
+</note>
+</compatibility>
 </eagle>
